File: Current Hacker/solder project.kicad_pcb (KiCad board)
At the start: 2 copper layers, 78.5 x 96 mm, 20 parts, among them J1 Conn_01x01_Pin, M1 Motor_DC, Q1 2N3904, Q2 2N3904, Q3 2N3904, SW1 SW_Push

Commit message: Add files via upload
Connections:
- M1 pad 1: Net-(M1-+) -> Net-(D1-A)
- M1 pad 2: Net-(BT1--) -> Net-(M1--)
- Q3 pad 1: Net-(M1-+) -> Net-(BT1--)
- Q3 pad 3: Net-(Q3-C) -> Net-(M1--)
- R1 pad 2: Net-(Q3-C) -> Net-(M1--)
- SW1 pad 1: Net-(D1-K) -> Net-(D1-A)
Routing:
- net Net-(D1-A): track 62.2 -> 248.7 mm, vias 0 -> 2
- net Net-(M1--): track 0.00 -> 99.0 mm, vias 0 -> 2
- net Net-(M1-+): track 83.9 -> 0.00 mm
- net Net-(BT1--): track 14.4 -> 74.7 mm
- net Net-(D1-K): track 59.8 -> 26.8 mm
- net Net-(Q3-C): track 11.8 -> 0.00 mm
